Commit message: Added missing tof sensors and cameras. Did not add the right position for cameras and tof sensors.
URDF worked!!

File: src/awdbot_description/urdf/rcjrobot.urdf.xacro (robot description, xacro)
@@ -12,12 +12,12 @@
   <xacro:property name="urdf_parameters" value="${xacro.load_yaml('$(find awdbot_description)/config/rcjrobot_params.yaml')}"/>
   <!-- Parse the parameters from the loaded configuration-array -->
-  <xacro:property name="wheel_radius" value="${urdf_parameters['wheel_radius']/1000}"/>
-  <xacro:property name="wheel_width" value="${urdf_parameters['wheel_width']/1000}"/>
-  <xacro:property name="wheel_mounting_offset_z" value="${urdf_parameters['wheel_mounting_offset_z']/1000}"/>
-  <xacro:property name="wheel_mounting_offset_x" value="${urdf_parameters['wheel_mounting_offset_x']/1000}"/>
-  <xacro:property name="wheel_clearance" value="${urdf_parameters['wheel_clearance']/1000}"/>
-  <xacro:property name="chassis_length" value="${urdf_parameters['chassis_length']/1000}"/>
-  <xacro:property name="chassis_width" value="${urdf_parameters['chassis_width']/1000}"/>
-  <xacro:property name="chassis_height" value="${urdf_parameters['chassis_height']/1000}"/>
+  <xacro:property name="wheel_radius" value="${urdf_parameters['wheel_radius']}"/>
+  <xacro:property name="wheel_width" value="${urdf_parameters['wheel_width']}"/>
+  <xacro:property name="wheel_mounting_offset_z" value="${urdf_parameters['wheel_mounting_offset_z']}"/>
+  <xacro:property name="wheel_mounting_offset_x" value="${urdf_parameters['wheel_mounting_offset_x']}"/>
+  <xacro:property name="wheel_clearance" value="${urdf_parameters['wheel_clearance']}"/>
+  <xacro:property name="chassis_length" value="${urdf_parameters['chassis_length']}"/>
+  <xacro:property name="chassis_width" value="${urdf_parameters['chassis_width']}"/>
+  <xacro:property name="chassis_height" value="${urdf_parameters['chassis_height']}"/>
   <!-- Constants -->
   <xacro:property name="MATH_PI" value="3.14159" />
@@ -31,5 +31,5 @@
   <xacro:include filename="$(find awdbot_description)/urdf/rcjrobot/wheels.urdf.xacro" />
   <!-- Add lidar -->
-  <xacro:include filename="$(find awdbot_description)/urdf/rcjrobot/lidar.urdf.xacro" />
+  <!-- <xacro:include filename="$(find awdbot_description)/urdf/rcjrobot/lidar.urdf.xacro" /> -->
   <!-- Add tof -->
   <!-- <xacro:include filename="$(find awdbot_description)/urdf/rcjrobot/tof.urdf.xacro" /> -->

File: src/awdbot_description/urdf/rcjrobot/camera.urdf.xacro (robot description, xacro)
@@ -1,79 +1,18 @@
 <?xml version="1.0"?>
-<robot xmlns:xacro="http://www.ros.org/wiki/xacro">
-    <!-- Parse the parameters from the loaded configuration-array -->
-    <xacro:property name="camera_height" value="0.006"/>
-    <xacro:property name="camera_diameter" value="0.004"/>
-    <xacro:property name="camera_link" value="camera_link"/>
-    <xacro:property name="camera_name" value="camera"/>
-    <xacro:property name="camera_topic" value="/camera/image_raw"/>
-    <xacro:property name="update_rate" value="10.0"/> <!--[Hz]-->
-    <xacro:property name="visualize" value="1"/>
-    <xacro:property name="horizontal_fov" value="1.21126"/>
-    <xacro:property name="image_width" value="640"/>
-    <xacro:property name="image_height" value="480"/>
-    <xacro:property name="image_format" value="RGB_INT8"/>
-    <xacro:property name="clip_near" value="0.1"/>
-    <xacro:property name="clip_far" value="100"/>
-    <xacro:property name="noise_stddev" value="0.007"/>
-    <!-- Add camera_mount -->
-    <link name="${camera_link}_mount_link">
-        <visual>
-            <origin xyz="0 0 ${camera_diameter / 2.0}" rpy="0 ${MATH_PI / 2.0} 0" />
-            <geometry>
-                <cylinder length="${camera_height}" radius="${camera_diameter / 2.0}"/>
-            </geometry>
-            <material name="green"/>
-        </visual>
-        <collision>
-            <origin xyz="0 0 ${camera_diameter / 2.0}" rpy="0 ${MATH_PI / 2.0} 0" />
-            <geometry>
-                <cylinder length="${camera_height}" radius="${camera_diameter / 2.0}"/>
-            </geometry>
-        </collision>
-        <inertial>
-            <mass value="0.01" />
-            <origin xyz="0 0 ${camera_diameter / 2.0}" rpy="0 0 0" />
-            <xacro:cylinder_inertia m="0.01" r="${camera_diameter / 2.0}" h="${camera_height}" />
-        </inertial>
-    </link>
-    <joint name="${camera_link}_mount_link_joint" type="fixed" >
-        <origin xyz="0.03 0 ${chassis_height / 2.0 - 0.02}" rpy="0 0 0" />
-        <parent link="base_link"/>
-        <child link="${camera_link}_mount_link" />
-    </joint>
-    <!-- Add camera_link -->
-    <link name="${camera_link}">
-    </link>
-    <joint name="${camera_link}_joint" type="fixed" >
-        <origin xyz="0 0 ${camera_diameter / 2.0}" rpy="0 0 0" />
-        <parent link="${camera_link}_mount_link"/>
-        <child link="${camera_link}" />
-    </joint>
-    <gazebo reference="${camera_link}">
-        <sensor name="${camera_name}" type="camera">
-            <pose relative_to='${camera_link}'>0 0 0 0 0 0</pose>
-            <always_on>1</always_on>
-            <update_rate>${update_rate}</update_rate>
-            <visualize>${visualize}</visualize>
-            <pose>0 0 0 0 0 0</pose>
-            <topic>${camera_topic}</topic>
-            <camera name="${camera_name}">
-                <horizontal_fov>${horizontal_fov}</horizontal_fov>
-                <image>
-                    <width>${image_width}</width>
-                    <height>${image_height}</height>
-                    <format>${image_format}</format>
-                </image>
-                <clip>
-                    <near>${clip_near}</near>
-                    <far>${clip_far}</far>
-                </clip>
-                <noise>
-                    <type>gaussian</type>
-                    <mean>0</mean>
-                    <stddev>${noise_stddev}</stddev>
-                </noise>
-            </camera>
-        </sensor>
-    </gazebo>
+<robot xmlns:xacro="http://ros.org/wiki/xacro">
+  <xacro:include filename="macros/camera.xacro"/>
+  <xacro:camera
+    name="left_camera"
+    parent="base_link"
+    xyz="0.2 0 0.1"
+    rpy="0 0 0"
+    chassis_height="${chassis_height}"
+  />
+  <xacro:camera
+    name="right_camera"
+    parent="base_link"
+    xyz="-0.2 0 0.1"
+    rpy="0 0 3.14"
+    chassis_height="${chassis_height}"
+  />
 </robot>

File: src/awdbot_description/urdf/rcjrobot/tof.urdf.xacro (robot description, xacro)
@@ -1,91 +1,12 @@
 <?xml version="1.0"?>
-<robot xmlns:xacro="http://www.ros.org/wiki/xacro">
-    <!-- Parse the parameters from the loaded configuration-array -->
-    <xacro:property name="lidar_height" value="0.004"/>
-    <xacro:property name="lidar_diameter" value="0.008"/>
-    <xacro:property name="lidar_link" value="tof_link"/>
-    <xacro:property name="lidar_name" value="tof_lidar"/>
-    <xacro:property name="lidar_topic" value="/tof_scan"/>
-    <xacro:property name="update_rate" value="20.0"/>
-    <xacro:property name="visualize" value="1"/>
-    <xacro:property name="h_samples" value="1"/>
-    <xacro:property name="h_res" value="1.0"/>
-    <xacro:property name="h_min_angle" value="${-1.0 / 180.0 * MATH_PI}"/>
-    <xacro:property name="h_max_angle" value="${1.0 / 180.0 * MATH_PI}"/>
-    <xacro:property name="v_samples" value="1.0"/>
-    <xacro:property name="v_res" value="1.0"/>
-    <xacro:property name="v_min_angle" value="0.0"/>
-    <xacro:property name="v_max_angle" value="0.0"/>
-    <xacro:property name="r_min" value="0.164"/>
-    <xacro:property name="r_max" value="12.0"/>
-    <xacro:property name="r_res" value="0.01"/>
-    <!-- Add lidar_mount -->
-    <link name="${lidar_link}_mount_link">
-        <visual>
-            <origin xyz="0 0 ${lidar_height / 2.0}" rpy="0 0 0" />
-            <geometry>
-                <cylinder length="${lidar_height}" radius="${lidar_diameter / 2.0}"/>
-            </geometry>
-            <material name="black"/>
-        </visual>
-        <collision>
-            <origin xyz="0 0 ${lidar_height / 2.0}" rpy="0 0 0" />
-            <geometry>
-                <cylinder length="${lidar_height}" radius="${lidar_diameter / 2.0}"/>
-            </geometry>
-        </collision>
-        <inertial>
-            <mass value="0.01" />
-            <origin xyz="0 0 ${lidar_height / 2.0}" rpy="0 0 0" />
-            <xacro:cylinder_inertia m="0.01" r="${lidar_diameter / 2.0}" h="${lidar_height}" />
-        </inertial>
-    </link>
-    <joint name="${lidar_link}_mount_link_joint" type="fixed" >
-        <origin xyz="0 0 ${chassis_height / 2.0}" rpy="0 0 0" />
-        <parent link="base_link"/>
-        <child link="${lidar_link}_mount_link" />
-    </joint>
-    <!-- Add lidar_link -->
-    <link name="${lidar_link}">
-    </link>
-    <joint name="${lidar_link}_joint" type="fixed" >
-        <origin xyz="0 0 ${lidar_height / 3.0 * 2.0}" rpy="0 0 0" />
-        <parent link="${lidar_link}_mount_link"/>
-        <child link="${lidar_link}" />
-    </joint>
-    <gazebo reference="${lidar_link}">
-        <sensor name="${lidar_name}" type="gpu_lidar">
-            <pose relative_to='${lidar_link}'>0 0 0 0 0 0</pose>
-            <topic>${lidar_topic}</topic>
-            <update_rate>${update_rate}</update_rate>
-            <visualize>${visualize}</visualize>
-            <always_on>true</always_on>
-            <ignition_frame_id>${lidar_link}</ignition_frame_id>
-            <gazebo_frame_id>${lidar_link}</gazebo_frame_id>
-            <frame_id>${lidar_link}</frame_id>
-            <gz_frame_id>${lidar_link}</gz_frame_id>
-            <ign_frame_id>${lidar_link}</ign_frame_id>
-            <lidar>
-                <scan>
-                    <horizontal>
-                        <samples>${h_samples}</samples>
-                        <resolution>${h_res}</resolution>
-                        <min_angle>${h_min_angle}</min_angle>
-                        <max_angle>${h_max_angle}</max_angle>
-                    </horizontal>
-                    <vertical>
-                        <samples>${v_samples}</samples>
-                        <resolution>${v_res}</resolution>
-                        <min_angle>${v_min_angle}</min_angle>
-                        <max_angle>${v_max_angle}</max_angle>
-                    </vertical>
-                </scan>
-                <range>
-                    <min>${r_min}</min>
-                    <max>${r_max}</max>
-                    <resolution>${r_res}</resolution>
-                </range>
-            </lidar>
-        </sensor>
-    </gazebo>
+<robot xmlns:xacro="http://ros.org/wiki/xacro">
+  <xacro:include filename="macros/tof.xacro"/>
+  <xacro:tof name="front_left_tof" parent="base_link" xyz="0.2 0 0.1" rpy="0 0 0"/>
+  <xacro:tof name="front_right_tof"  parent="base_link" xyz="-0.2 0 0.1" rpy="0 0 3.14"/>
+  <xacro:tof name="left_front_tof"  parent="base_link" xyz="-0.2 0 0.1" rpy="0 0 3.14"/>
+  <xacro:tof name="left_rear_tof"  parent="base_link" xyz="-0.2 0 0.1" rpy="0 0 3.14"/>
+  <xacro:tof name="right_front_tof"  parent="base_link" xyz="-0.2 0 0.1" rpy="0 0 3.14"/>
+  <xacro:tof name="right_rear_tof"  parent="base_link" xyz="-0.2 0 0.1" rpy="0 0 3.14"/>
+  <xacro:tof name="rear_left_tof"  parent="base_link" xyz="-0.2 0 0.1" rpy="0 0 3.14"/>
+  <xacro:tof name="rear_right_tof"  parent="base_link" xyz="-0.2 0 0.1" rpy="0 0 3.14"/>
 </robot>

File: src/awdbot_description/urdf/rcjrobot/wheels.urdf.xacro (robot description, xacro)
@@ -1,139 +1,40 @@
 <?xml version="1.0"?>
 <robot xmlns:xacro="http://www.ros.org/wiki/xacro">
-    <!-- Add wheel_front_left_mount to base_link -->
-    <link name="wheel_front_left_mount">
-    </link>
-    <joint name="wheel_front_left_mount_joint" type="fixed" >
-        <origin xyz="${wheel_mounting_offset_x} ${chassis_width / 2.0} ${- chassis_height / 2 + wheel_mounting_offset_z}" rpy="0 0 0" />
-        <parent link="base_link"/>
-        <child link="wheel_front_left_mount" />
-    </joint>
-    <!-- Add wheel_front_left to wheel_front_left_mount -->
-    <link name="wheel_front_left">
-        <visual>
-            <origin xyz="0 0 0" rpy="0 0 0" />
-            <geometry>
-                <mesh filename="file://$(find awdbot_description)/meshes/left_wheel.dae" scale="0.001 0.001 0.001" />
-            </geometry>
-        </visual>
-        <collision>
-            <origin xyz="0 0 0" rpy="${MATH_PI/2} 0 0" />
-            <geometry>
-                <cylinder length="${wheel_width}" radius="${wheel_radius}"/>
-            </geometry>
-        </collision>
-        <inertial>
-            <mass value="5.0" />
-            <origin xyz="0 0 0" rpy="${MATH_PI/2} 0 0" />
-            <xacro:cylinder_inertia m="5.0" r="${wheel_radius}" h="${wheel_width}" />
-        </inertial>
-    </link>
-    <joint name="wheel_front_left_joint" type="continuous">
-        <parent link="wheel_front_left_mount"/>
-        <child link="wheel_front_left"/>
-        <axis xyz="0 1 0"/>
-        <origin xyz="0 0 0"/>
-    </joint>
-    <!-- Add wheel_front_right_mount to base_link -->
-    <link name="wheel_front_right_mount">
-    </link>
-    <joint name="wheel_front_right_mount_joint" type="fixed" >
-        <origin xyz="${wheel_mounting_offset_x} ${- chassis_width / 2.0} ${-chassis_height / 2 + wheel_mounting_offset_z}" rpy="0 0 0" />
-        <parent link="base_link"/>
-        <child link="wheel_front_right_mount" />
-    </joint>
-    <!-- Add wheel_front_right to wheel_front_right_mount -->
-    <link name="wheel_front_right">
-        <visual>
-            <origin xyz="0 0 0" rpy="0 0 0" />
-            <geometry>
-                <mesh filename="file://$(find awdbot_description)/meshes/right_wheel.dae" scale="0.001 0.001 0.001" />
-            </geometry>
-        </visual>
-        <collision>
-            <origin xyz="0 0 0" rpy="${MATH_PI/2} 0 0" />
-            <geometry>
-                <cylinder length="${wheel_width}" radius="${wheel_radius}"/>
-            </geometry>
-        </collision>
-        <inertial>
-            <mass value="5.0" />
-            <origin xyz="0 0 0" rpy="${MATH_PI/2} 0 0" />
-            <xacro:cylinder_inertia m="5.0" r="${wheel_radius}" h="${wheel_width}" />
-        </inertial>
-    </link>
-    <joint name="wheel_front_right_joint" type="continuous">
-        <parent link="wheel_front_right_mount"/>
-        <child link="wheel_front_right"/>
-        <axis xyz="0 1 0"/>
-        <origin xyz="0 0 0"/>
-    </joint>
-    <!-- Add wheel_rear_left_mount to base_link -->
-    <link name="wheel_rear_left_mount">
-    </link>
-    <joint name="wheel_rear_left_mount_joint" type="fixed" >
-        <origin xyz="${- wheel_mounting_offset_x} ${chassis_width / 2.0} ${-chassis_height / 2 + wheel_mounting_offset_z}" rpy="0 0 0" />
-        <parent link="base_link"/>
-        <child link="wheel_rear_left_mount" />
-    </joint>
-    <!-- Add wheel_rear_left to wheel_rear_left_mount -->
-    <link name="wheel_rear_left">
-        <visual>
-            <origin xyz="0 0 0" rpy="0 0 0" />
-            <geometry>
-                <mesh filename="file://$(find awdbot_description)/meshes/left_wheel.dae" scale="0.001 0.001 0.001" />
-            </geometry>
-        </visual>
-        <collision>
-            <origin xyz="0 0 0" rpy="${MATH_PI/2} 0 0" />
-            <geometry>
-                <cylinder length="${wheel_width}" radius="${wheel_radius}"/>
-            </geometry>
-        </collision>
-        <inertial>
-            <mass value="5.0" />
-            <origin xyz="0 0 0" rpy="${MATH_PI/2} 0 0" />
-            <xacro:cylinder_inertia m="5.0" r="${wheel_radius}" h="${wheel_width}" />
-        </inertial>
-    </link>
-    <joint name="wheel_rear_left_joint" type="continuous">
-        <parent link="wheel_rear_left_mount"/>
-        <child link="wheel_rear_left"/>
-        <axis xyz="0 1 0"/>
-        <origin xyz="0 0 0"/>
-    </joint>
-    <!-- Add wheel_rear_right_mount to base_link -->
-    <link name="wheel_rear_right_mount">
-    </link>
-    <joint name="wheel_rear_right_mount_joint" type="fixed" >
-        <origin xyz="${- wheel_mounting_offset_x} ${- chassis_width / 2.0} ${- chassis_height / 2 + wheel_mounting_offset_z}" rpy="0 0 0" />
-        <parent link="base_link"/>
-        <child link="wheel_rear_right_mount" />
-    </joint>
-    <!-- Add wheel_rear_right to wheel_rear_right_mount -->
-    <link name="wheel_rear_right">
-        <visual>
-            <origin xyz="0 0 0" rpy="0 0 0" />
-            <geometry>
-                <mesh filename="file://$(find awdbot_description)/meshes/right_wheel.dae" scale="0.001 0.001 0.001" />
-            </geometry>
-        </visual>
-        <collision>
-            <origin xyz="0 0 0" rpy="${MATH_PI/2} 0 0" />
-            <geometry>
-                <cylinder length="${wheel_width}" radius="${wheel_radius}"/>
-            </geometry>
-        </collision>
-        <inertial>
-            <mass value="5.0" />
-            <origin xyz="0 0 0" rpy="${MATH_PI/2} 0 0" />
-            <xacro:cylinder_inertia m="5.0" r="${wheel_radius}" h="${wheel_width}" />
-        </inertial>
-    </link>
-    <joint name="wheel_rear_right_joint" type="continuous">
-        <parent link="wheel_rear_right_mount"/>
-        <child link="wheel_rear_right"/>
-        <axis xyz="0 1 0"/>
-        <origin xyz="0 0 0"/>
-    </joint>
+    <xacro:include filename="macros/wheels.xacro"/>
+    <xacro:wheel
+        name="wheel_front_left"
+        parent="base_link"
+        xyz="${wheel_mounting_offset_x} ${chassis_width / 2.0} ${-chassis_height / 2 + wheel_mounting_offset_z}"
+        rpy="0 0 0"
+        visual_rpy="0 0 0"
+        wheel_radius="${wheel_radius}"
+        wheel_width="${wheel_width}"
+    />
+    <xacro:wheel
+        name="wheel_front_right"
+        parent="base_link"
+        xyz="${wheel_mounting_offset_x} ${-chassis_width / 2.0} ${-chassis_height / 2 + wheel_mounting_offset_z}"
+        rpy="0 0 0"
+        visual_rpy="0 0 0"
+        wheel_radius="${wheel_radius}"
+        wheel_width="${wheel_width}"
+    />
+    <xacro:wheel
+        name="wheel_rear_left"
+        parent="base_link"
+        xyz="${-wheel_mounting_offset_x} ${chassis_width / 2.0} ${-chassis_height / 2 + wheel_mounting_offset_z}"
+        rpy="0 0 0"
+        visual_rpy="0 0 0"
+        wheel_radius="${wheel_radius}"
+        wheel_width="${wheel_width}"
+    />
+    <xacro:wheel
+        name="wheel_rear_right"
+        parent="base_link"
+        xyz="${-wheel_mounting_offset_x} ${-chassis_width / 2.0} ${-chassis_height / 2 + wheel_mounting_offset_z}"
+        rpy="0 0 0"
+        visual_rpy="0 0 0"
+        wheel_radius="${wheel_radius}"
+        wheel_width="${wheel_width}"
+    />
 </robot>
