Commit message: Added TOF Sensor and cameras to URDF

File: src/awdbot_description/urdf/rcjrobot.urdf.xacro (robot description, xacro)
@@ -33,5 +33,5 @@
   <!-- <xacro:include filename="$(find awdbot_description)/urdf/rcjrobot/lidar.urdf.xacro" /> -->
   <!-- Add tof -->
-  <!-- <xacro:include filename="$(find awdbot_description)/urdf/rcjrobot/tof.urdf.xacro" /> -->
+  <xacro:include filename="$(find awdbot_description)/urdf/rcjrobot/tof.urdf.xacro" />
   <!-- Add camera -->
   <xacro:include filename="$(find awdbot_description)/urdf/rcjrobot/camera.urdf.xacro" />

File: src/awdbot_description/urdf/rcjrobot/camera.urdf.xacro (robot description, xacro)
@@ -5,6 +5,6 @@
     name="left_camera"
     parent="base_link"
-    xyz="0.2 0 0.1"
-    rpy="0 0 0"
+    xyz="-0.01 0.04 0.04"
+    rpy="0 0 ${MATH_PI/2}"
     chassis_height="${chassis_height}"
   />
@@ -12,6 +12,6 @@
     name="right_camera"
     parent="base_link"
-    xyz="-0.2 0 0.1"
-    rpy="0 0 3.14"
+    xyz="-0.01 -0.04 0.04"
+    rpy="0 0 ${-MATH_PI/2}"
     chassis_height="${chassis_height}"
   />

File: src/awdbot_description/urdf/rcjrobot/macros/camera.xacro (robot description, xacro)
@@ -5,7 +5,7 @@
         <xacro:property name="camera_height" value="0.006"/>
         <xacro:property name="camera_diameter" value="0.004"/>
-        <xacro:property name="camera_link" value="${name}_camera_link"/>
-        <xacro:property name="camera_name" value="${name}_camera"/>
-        <xacro:property name="camera_topic" value="/${name}_camera/image_raw"/>
+        <xacro:property name="camera_link" value="${name}_link"/>
+        <xacro:property name="camera_name" value="${name}"/>
+        <xacro:property name="camera_topic" value="/${name}/image_raw"/>
         <xacro:property name="update_rate" value="10.0"/> <!--[Hz]-->
         <xacro:property name="visualize" value="1"/>
@@ -18,7 +18,7 @@
         <xacro:property name="noise_stddev" value="0.007"/>
         <!-- Add camera_mount -->
-        <link name="${camera_link}_mount_link">
+        <link name="${name}_mount_link">
             <visual>
-                <origin xyz="0 0 ${camera_diameter / 2.0}" rpy="0 ${MATH_PI / 2.0} 0" />
+                <origin xyz="0 0 0" rpy="0 0 0" />
                 <geometry>
                     <cylinder length="${camera_height}" radius="${camera_diameter / 2.0}"/>
@@ -27,5 +27,5 @@
             </visual>
             <collision>
-                <origin xyz="0 0 ${camera_diameter / 2.0}" rpy="0 ${MATH_PI / 2.0} 0" />
+                <origin xyz="0 0 0" rpy="0 0 0" />
                 <geometry>
                     <cylinder length="${camera_height}" radius="${camera_diameter / 2.0}"/>
@@ -34,24 +34,24 @@
             <inertial>
                 <mass value="0.01" />
-                <origin xyz="0 0 ${camera_diameter / 2.0}" rpy="0 0 0" />
+                <origin xyz="0 0 0" rpy="0 0 0" />
                 <xacro:cylinder_inertia m="0.01" r="${camera_diameter / 2.0}" h="${camera_height}" />
             </inertial>
         </link>
-        <joint name="${camera_link}_mount_link_joint" type="fixed" >
-            <origin xyz="0.03 0 ${chassis_height / 2.0 - 0.02}" rpy="0 0 0" />
+        <joint name="${name}_mount_link_joint" type="fixed" >
+            <origin xyz="${xyz}" rpy="${rpy}" />
             <parent link="base_link"/>
-            <child link="${camera_link}_mount_link" />
+            <child link="${name}_mount_link" />
         </joint>
-        <!-- Add camera_link -->
-        <link name="${camera_link}">
+        <!-- Add name -->
+        <link name="${name}">
         </link>
-        <joint name="${camera_link}_joint" type="fixed" >
-            <origin xyz="0 0 ${camera_diameter / 2.0}" rpy="0 0 0" />
-            <parent link="${camera_link}_mount_link"/>
-            <child link="${camera_link}" />
+        <joint name="${name}_joint" type="fixed" >
+            <origin xyz="0 0 0" rpy="0 0 0"/>
+            <parent link="${name}_mount_link"/>
+            <child link="${name}" />
         </joint>
-        <gazebo reference="${camera_link}">
+        <gazebo reference="${name}">
             <sensor name="${camera_name}" type="camera">
-                <pose relative_to='${camera_link}'>0 0 0 0 0 0</pose>
+                <pose relative_to='${name}'>0 0 0 0 0 0</pose>
                 <always_on>1</always_on>
                 <update_rate>${update_rate}</update_rate>

File: src/awdbot_description/urdf/rcjrobot/macros/tof.xacro (robot description, xacro)
@@ -1,5 +1,5 @@
 <?xml version="1.0"?>
 <robot xmlns:xacro="http://www.ros.org/wiki/xacro">
-    <xacro:macro name="tof" params="name parent xyz rpy chassis_height">
+    <xacro:macro name="tof" params="name parent xyz rpy">
         <!-- Parse the parameters from the loaded configuration-array -->
         <xacro:property name="lidar_height" value="0.004"/>
@@ -12,11 +12,11 @@
         <xacro:property name="h_samples" value="1"/>
         <xacro:property name="h_res" value="1.0"/>
-        <xacro:property name="h_min_angle" value="${-1.0 / 180.0 * MATH_PI}"/>
-        <xacro:property name="h_max_angle" value="${1.0 / 180.0 * MATH_PI}"/>
-        <xacro:property name="v_samples" value="1.0"/>
+        <xacro:property name="h_min_angle" value="0.01"/>
+        <xacro:property name="h_max_angle" value="0.01"/>
+        <xacro:property name="v_samples" value="1"/>
         <xacro:property name="v_res" value="1.0"/>
         <xacro:property name="v_min_angle" value="0.0"/>
         <xacro:property name="v_max_angle" value="0.0"/>
-        <xacro:property name="r_min" value="0.164"/>
+        <xacro:property name="r_min" value="0.04"/>
         <xacro:property name="r_max" value="12.0"/>
         <xacro:property name="r_res" value="0.01"/>
@@ -42,14 +42,14 @@
             </inertial>
         </link>
-        <joint name="${name}_mount_link_joint" type="fixed" >
+        <joint name="${name}_mount_joint" type="fixed" >
             <origin xyz="${xyz}" rpy="${rpy}" />
             <parent link="${parent}"/>
             <child link="${name}_mount_link" />
         </joint>
-        <!-- Add lidar_link -->
+        <!-- Add name -->
         <link name="${name}">
         </link>
         <joint name="${name}_joint" type="fixed" >
-            <origin xyz="0 0 0}" rpy="0 0 0" />
+            <origin xyz="0 0 0" rpy="0 0 0" />
             <parent link="${name}_mount_link"/>
             <child link="${name}" />
@@ -62,9 +62,9 @@
                 <visualize>${visualize}</visualize>
                 <always_on>true</always_on>
-                <ignition_frame_id>${lidar_link}</ignition_frame_id>
-                <gazebo_frame_id>${lidar_link}</gazebo_frame_id>
-                <frame_id>${lidar_link}</frame_id>
-                <gz_frame_id>${lidar_link}</gz_frame_id>
-                <ign_frame_id>${lidar_link}</ign_frame_id>
+                <ignition_frame_id>${name}</ignition_frame_id>
+                <gazebo_frame_id>${name}</gazebo_frame_id>
+                <frame_id>${name}</frame_id>
+                <gz_frame_id>${name}</gz_frame_id>
+                <ign_frame_id>${name}</ign_frame_id>
                 <lidar>
                     <scan>

File: src/awdbot_description/urdf/rcjrobot/macros/wheels.xacro (robot description, xacro)
@@ -11,5 +11,5 @@
         <link name="${name}">
             <visual>
-                <origin xyz="0 0 0" rpy="0 0 0" />
+                <origin xyz="0 0 0" rpy="${visual_rpy}" />
                 <geometry>
                     <mesh filename="file://$(find awdbot_description)/meshes/wheel.dae" scale="0.001 0.001 0.001" />
@@ -28,7 +28,7 @@
             </inertial>
         </link>
-        <joint name="${wheel_width}_joint" type="continuous">
-            <parent link="${wheel_width}_mount"/>
-            <child link="${wheel_width}"/>
+        <joint name="${name}_joint" type="continuous">
+            <parent link="${name}_mount"/>
+            <child link="${name}"/>
             <axis xyz="0 1 0"/>
             <origin xyz="0 0 0"/>

File: src/awdbot_description/urdf/rcjrobot/tof.urdf.xacro (robot description, xacro)
@@ -2,11 +2,12 @@
 <robot xmlns:xacro="http://ros.org/wiki/xacro">
   <xacro:include filename="macros/tof.xacro"/>
-  <xacro:tof name="front_left_tof" parent="base_link" xyz="0.2 0 0.1" rpy="0 0 0"/>
-  <xacro:tof name="front_right_tof"  parent="base_link" xyz="-0.2 0 0.1" rpy="0 0 3.14"/>
-  <xacro:tof name="left_front_tof"  parent="base_link" xyz="-0.2 0 0.1" rpy="0 0 3.14"/>
-  <xacro:tof name="left_rear_tof"  parent="base_link" xyz="-0.2 0 0.1" rpy="0 0 3.14"/>
-  <xacro:tof name="right_front_tof"  parent="base_link" xyz="-0.2 0 0.1" rpy="0 0 3.14"/>
-  <xacro:tof name="right_rear_tof"  parent="base_link" xyz="-0.2 0 0.1" rpy="0 0 3.14"/>
-  <xacro:tof name="rear_left_tof"  parent="base_link" xyz="-0.2 0 0.1" rpy="0 0 3.14"/>
-  <xacro:tof name="rear_right_tof"  parent="base_link" xyz="-0.2 0 0.1" rpy="0 0 3.14"/>
+  <!-- Maße vom base_link weg, der sich in der mitte des chassis befindet -->
+  <xacro:tof name="front_left_tof" parent="base_link" xyz="0.045 0.0312 0.016" rpy="0 0 0"/>
+  <xacro:tof name="front_right_tof"  parent="base_link" xyz="0.045 -0.0312 0.016" rpy="0 0 0"/>
+  <xacro:tof name="left_front_tof"  parent="base_link" xyz="0.0226 0.0325 0.03" rpy="0 0 0"/>
+  <xacro:tof name="left_rear_tof"  parent="base_link" xyz="-0.0465 0.02 0.03" rpy="0 0 0"/>
+  <xacro:tof name="right_front_tof"  parent="base_link" xyz="0.0226 -0.0325 0.03" rpy="0 0 0"/>
+  <xacro:tof name="right_rear_tof"  parent="base_link" xyz="-0.0465 -0.02 0.034" rpy="0 0 0"/>
+  <xacro:tof name="rear_left_tof"  parent="base_link" xyz="-0.0765 0.046 -0.01914" rpy="0 0 0"/>
+  <xacro:tof name="rear_right_tof"  parent="base_link" xyz="-0.0765 -0.046 -0.01914" rpy="0 0 0"/>
 </robot>

File: src/awdbot_description/urdf/rcjrobot/wheels.urdf.xacro (robot description, xacro)
@@ -1,4 +1,4 @@
 <?xml version="1.0"?>
-<robot xmlns:xacro="http://www.ros.org/wiki/xacro">
+<robot xmlns:xacro="http://ros.org/wiki/xacro">
     <xacro:include filename="macros/wheels.xacro"/>
     <xacro:wheel
@@ -7,5 +7,5 @@
         xyz="${wheel_mounting_offset_x} ${chassis_width / 2.0} ${-chassis_height / 2 + wheel_mounting_offset_z}"
         rpy="0 0 0"
-        visual_rpy="0 0 0"
+        visual_rpy="0 0 ${MATH_PI}"
         wheel_radius="${wheel_radius}"
         wheel_width="${wheel_width}"
@@ -25,5 +25,5 @@
         xyz="${-wheel_mounting_offset_x} ${chassis_width / 2.0} ${-chassis_height / 2 + wheel_mounting_offset_z}"
         rpy="0 0 0"
-        visual_rpy="0 0 0"
+        visual_rpy="0 0 ${MATH_PI}"
         wheel_radius="${wheel_radius}"
         wheel_width="${wheel_width}"
